Commit message: added a mock launch file and modified the files to have the 140 gripper as the default since that is the one we bought

File: robotiq_description/urdf/robotiq_2f_140_gripper.urdf.xacro (robot description, xacro)
@@ -3,8 +3,9 @@
     <!-- parameters -->
     <xacro:arg name="use_fake_hardware" default="true" />
+    <xacro:arg name="parent" default="world" />
     <!-- Import macros -->
     <xacro:include filename="$(find robotiq_description)/urdf/robotiq_2f_140_macro.urdf.xacro" />
-    <link name="world" />
-    <xacro:robotiq_gripper name="RobotiqGripperHardwareInterface" prefix="" parent="world" use_fake_hardware="$(arg use_fake_hardware)">
+    <link name="$(arg parent)" />
+    <xacro:robotiq_gripper name="RobotiqGripperHardwareInterface" prefix="" parent="$(arg parent)" use_fake_hardware="$(arg use_fake_hardware)">
         <origin xyz="0 0 0" rpy="0 0 0" />
     </xacro:robotiq_gripper>
